File: 433_Antenna/433_Antenna.sch (KiCad schematic (older format))
At the start: 15 parts

Commit message: Small changes
Parts:
- gave numbers to parts that had none: 15
Changed lines of the file:
@@
 $EndDescr
 $Comp
-L Device:C C?
+L Device:C C101
 U 1 1 5DAD2CEA
 P 2825 1750
-F 0 "C?" H 2940 1796 50  0000 L CNN
+F 0 "C101" H 2940 1796 50  0000 L CNN
 F 1 "C" H 2940 1705 50  0000 L CNN
 F 2 "Capacitor_SMD:C_0402_1005Metric" H 2863 1600 50  0001 C CNN
@@
 $EndComp
 $Comp
-L pspice:INDUCTOR L?
+L pspice:INDUCTOR L101
 U 1 1 5DAD324F
 P 3225 1600
-F 0 "L?" H 3225 1815 50  0000 C CNN
+F 0 "L101" H 3225 1815 50  0000 C CNN
 F 1 "INDUCTOR" H 3225 1724 50  0000 C CNN
 F 2 "Capacitor_SMD:C_0402_1005Metric" H 3225 1600 50  0001 C CNN
@@
 $EndComp
 $Comp
-L Device:C C?
+L Device:C C104
 U 1 1 5DAD3534
 P 3600 1750
-F 0 "C?" H 3715 1796 50  0000 L CNN
+F 0 "C104" H 3715 1796 50  0000 L CNN
 F 1 "C" H 3715 1705 50  0000 L CNN
 F 2 "Capacitor_SMD:C_0402_1005Metric" H 3638 1600 50  0001 C CNN
@@
 $EndComp
 $Comp
-L Connector:Conn_Coaxial J?
+L Connector:Conn_Coaxial J101
 U 1 1 5DAD5293
 P 2025 1600
-F 0 "J?" H 1953 1838 50  0000 C CNN
+F 0 "J101" H 1953 1838 50  0000 C CNN
 F 1 "Conn_Coaxial" H 1953 1747 50  0000 C CNN
 F 2 "Connector_Coaxial:SMA_Amphenol_132134-11_Vertical" H 2025 1600 50  0001 C CNN
@@
 Connection ~ 2825 2250
 $Comp
-L power:GND #PWR?
+L power:GND #PWR0101
 U 1 1 5DAD6455
 P 3075 2375
-F 0 "#PWR?" H 3075 2125 50  0001 C CNN
+F 0 "#PWR0101" H 3075 2125 50  0001 C CNN
 F 1 "GND" H 3080 2202 50  0000 C CNN
 F 2 "" H 3075 2375 50  0001 C CNN
@@
 	3075 2250 2825 2250
 $Comp
-L Device:Antenna AE?
+L Device:Antenna AE101
 U 1 1 5DAD7A90
 P 4025 1150
-F 0 "AE?" H 4105 1139 50  0000 L CNN
+F 0 "AE101" H 4105 1139 50  0000 L CNN
 F 1 "Antenna" H 4105 1048 50  0000 L CNN
 F 2 "MeanderAntenna:0p8x" H 4025 1150 50  0001 C CNN
@@
 	4025 1350 4025 1600
 $Comp
-L Device:C C?
+L Device:C C102
 U 1 1 5DF20F9D
 P 2850 3500
-F 0 "C?" H 2965 3546 50  0000 L CNN
+F 0 "C102" H 2965 3546 50  0000 L CNN
 F 1 "C" H 2965 3455 50  0000 L CNN
 F 2 "Capacitor_SMD:C_0402_1005Metric" H 2888 3350 50  0001 C CNN
@@
 $EndComp
 $Comp
-L pspice:INDUCTOR L?
+L pspice:INDUCTOR L102
 U 1 1 5DF20FA3
 P 3250 3350
-F 0 "L?" H 3250 3565 50  0000 C CNN
+F 0 "L102" H 3250 3565 50  0000 C CNN
 F 1 "INDUCTOR" H 3250 3474 50  0000 C CNN
 F 2 "Capacitor_SMD:C_0402_1005Metric" H 3250 3350 50  0001 C CNN
@@
 $EndComp
 $Comp
-L Device:C C?
+L Device:C C105
 U 1 1 5DF20FA9
 P 3625 3500
-F 0 "C?" H 3740 3546 50  0000 L CNN
+F 0 "C105" H 3740 3546 50  0000 L CNN
 F 1 "C" H 3740 3455 50  0000 L CNN
 F 2 "Capacitor_SMD:C_0402_1005Metric" H 3663 3350 50  0001 C CNN
@@
 $EndComp
 $Comp
-L Connector:Conn_Coaxial J?
+L Connector:Conn_Coaxial J102
 U 1 1 5DF20FAF
 P 2050 3350
-F 0 "J?" H 1978 3588 50  0000 C CNN
+F 0 "J102" H 1978 3588 50  0000 C CNN
 F 1 "Conn_Coaxial" H 1978 3497 50  0000 C CNN
 F 2 "Connector_Coaxial:SMA_Amphenol_132134-11_Vertical" H 2050 3350 50  0001 C CNN
@@
 Connection ~ 2850 4000
 $Comp
-L power:GND #PWR?
+L power:GND #PWR0102
 U 1 1 5DF20FC1
 P 3100 4125
-F 0 "#PWR?" H 3100 3875 50  0001 C CNN
+F 0 "#PWR0102" H 3100 3875 50  0001 C CNN
 F 1 "GND" H 3105 3952 50  0000 C CNN
 F 2 "" H 3100 4125 50  0001 C CNN
@@
 	3100 4000 2850 4000
 $Comp
-L Device:Antenna AE?
+L Device:Antenna AE102
 U 1 1 5DF20FCA
 P 4050 2900
-F 0 "AE?" H 4130 2889 50  0000 L CNN
+F 0 "AE102" H 4130 2889 50  0000 L CNN
 F 1 "Antenna" H 4130 2798 50  0000 L CNN
 F 2 "MeanderAntenna:1" H 4050 2900 50  0001 C CNN
@@
 	4050 3100 4050 3350
 $Comp
-L Device:C C?
+L Device:C C103
 U 1 1 5DF2277A
 P 2950 5250
-F 0 "C?" H 3065 5296 50  0000 L CNN
+F 0 "C103" H 3065 5296 50  0000 L CNN
 F 1 "C" H 3065 5205 50  0000 L CNN
 F 2 "Capacitor_SMD:C_0402_1005Metric" H 2988 5100 50  0001 C CNN
@@
 $EndComp
 $Comp
-L pspice:INDUCTOR L?
+L pspice:INDUCTOR L103
 U 1 1 5DF22780
 P 3350 5100
-F 0 "L?" H 3350 5315 50  0000 C CNN
+F 0 "L103" H 3350 5315 50  0000 C CNN
 F 1 "INDUCTOR" H 3350 5224 50  0000 C CNN
 F 2 "Capacitor_SMD:C_0402_1005Metric" H 3350 5100 50  0001 C CNN
@@
 $EndComp
 $Comp
-L Device:C C?
+L Device:C C106
 U 1 1 5DF22786
 P 3725 5250
-F 0 "C?" H 3840 5296 50  0000 L CNN
+F 0 "C106" H 3840 5296 50  0000 L CNN
 F 1 "C" H 3840 5205 50  0000 L CNN
 F 2 "Capacitor_SMD:C_0402_1005Metric" H 3763 5100 50  0001 C CNN
@@
 $EndComp
 $Comp
-L Connector:Conn_Coaxial J?
+L Connector:Conn_Coaxial J103
 U 1 1 5DF2278C
 P 2150 5100
-F 0 "J?" H 2078 5338 50  0000 C CNN
+F 0 "J103" H 2078 5338 50  0000 C CNN
 F 1 "Conn_Coaxial" H 2078 5247 50  0000 C CNN
 F 2 "Connector_Coaxial:SMA_Amphenol_132134-11_Vertical" H 2150 5100 50  0001 C CNN
@@
 Connection ~ 2950 5750
 $Comp
-L power:GND #PWR?
+L power:GND #PWR0103
 U 1 1 5DF2279E
 P 3200 5875
-F 0 "#PWR?" H 3200 5625 50  0001 C CNN
+F 0 "#PWR0103" H 3200 5625 50  0001 C CNN
 F 1 "GND" H 3205 5702 50  0000 C CNN
 F 2 "" H 3200 5875 50  0001 C CNN
@@
 	3200 5750 2950 5750
 $Comp
-L Device:Antenna AE?
+L Device:Antenna AE103
 U 1 1 5DF227A7
 P 4150 4650
-F 0 "AE?" H 4230 4639 50  0000 L CNN
+F 0 "AE103" H 4230 4639 50  0000 L CNN
 F 1 "Antenna" H 4230 4548 50  0000 L CNN
 F 2 "MeanderAntenna:1p2x" H 4150 4650 50  0001 C CNN
